File: EuroESP32.brd (EAGLE design)
At the start: 30 x 108 mm, 117 parts, among them IC1 TL074D, IC10 MCP6004, IC2 TL072, IC3 TL072, IC4 WM8731, IC5 TL074D, IC7 ADP7118, P4 POWER_SIMPLE10, U1 LM4040SOT23, U2 MCP3204-CI/SL

Commit message: Update EuroESP32.brd
Parts:
- moved C6 22.9 mm to (21.0, 17.5), turned to 180 degrees
- moved C1 18.5 mm to (22.7, 7.84), turned to 180 degrees
- moved REGULATOR 2.94 mm to (26.3, 15.1), turned to 0 degrees
- moved C34 1.40 mm to (26.6, 22.5)
- moved +12V 1.40 mm to (2.93, 47.3), turned to 0 degrees
- moved +3.3VA 1.40 mm to (2.93, 49.8), turned to 0 degrees
- moved -10VREF 1.40 mm to (2.93, 39.6), turned to 0 degrees
- moved -12V 1.40 mm to (2.93, 42.2), turned to 0 degrees
- moved CVIN(100K)0 1.40 mm to (2.93, 26.9), turned to 0 degrees
- moved CVIN(100K)1 1.40 mm to (2.93, 24.4), turned to 0 degrees
- moved CVIN(100K)2 1.40 mm to (2.93, 21.9), turned to 0 degrees
- moved CVIN(100K)3 1.40 mm to (2.93, 19.3), turned to 0 degrees
- moved CVOUT1 1.40 mm to (2.93, 16.8), turned to 0 degrees
- moved CVOUT2 1.40 mm to (2.93, 14.2), turned to 0 degrees
- moved CVOUT3 1.40 mm to (2.93, 11.7), turned to 0 degrees
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Routing:
- net +3.3VA: track 131.6 -> 322.3 mm, vias 2 -> 5
- net -12V: track 60.2 -> 149.2 mm
- net N$1: track 0.00 -> 51.8 mm
- net N$25: track 0.00 -> 42.8 mm
- net -10VREF: track 20.9 -> 59.4 mm, vias 0 -> 1
- net N$2: track 0.00 -> 35.8 mm
- net GND: track 378.9 -> 406.9 mm, vias 8 -> 9
- net N$46: track 4.25 -> 28.7 mm
- net N$29: track 0.00 -> 21.1 mm
- net 5V: track 86.7 -> 98.7 mm
- net +12V: track 122.2 -> 132.5 mm, vias 1 -> 2
- net N$15: track 57.5 -> 54.7 mm
- net N$19: track 18.4 -> 15.6 mm
- net N$21: track 54.3 -> 51.9 mm
- net N$17: track 31.0 -> 29.0 mm
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